File: dsky/dsky-7seg.sch (KiCad schematic (older format))
At the start: 40 parts, among them Q1 PMOS, Q2 PMOS, Q3 PMOS, Q4 PMOS, Q5 PMOS, Q6 PMOS, Q7 PMOS, Q8 PMOS, U10 HDSP-7403, U11 HDSP-7403, U12 HDSP-7403, U13 HDSP-7403, U14 HDSP-7403, U15 HDSP-7403, U16 HDSP-7403, U17 HDSP-7403, U18 ULN2003, U19 HDSP-7403, U2 HDSP-7403, U20 HDSP-7403, U21 HDSP-7403, U22 HDSP-7403, U23 HDSP-7403, U24 ULN2003, U25 ULN2003, U3 HDSP-7403, U4 HDSP-7403, U5 HDSP-7403, U6 HDSP-7403, U7 HDSP-7403, U8 HDSP-7403, U9 HDSP-7403

Commit message: this hard drive is dying
Parts:
- added R13, R14, R15, R16, R20, R34, R36, R37: 1K, Resistor_SMD:R_0402_1005Metric, symbol Device:R
Connections:
- net +3V3: now also R13.2, R14.2, R15.2, R16.2, R20.2, R34.2, R36.2, R37.2
- net MCU_7SEG_A: now also R37.1
- net MCU_7SEG_B: now also R36.1
- net MCU_7SEG_C: now also R34.1
- net MCU_7SEG_D: now also R20.1
- net MCU_7SEG_DP: now also R13.1
- net MCU_7SEG_E: now also R16.1
- net MCU_7SEG_F: now also R15.1
- net MCU_7SEG_G: now also R14.1
Changed lines of the file:
@@
 AR Path="/62EB4C8F/62FD0741" Ref="Q3"  Part="1"
 F 0 "Q3" V 9300 2050 50  0000 L CNN
-F 1 "PMOS" V 9150 1750 50  0000 L CNN
+F 1 "PMOS" V 9200 1750 50  0000 L CNN
 F 2 "Package_TO_SOT_SMD:SOT-23" H 9600 2100 50  0001 C CNN
 F 3 "~" H 9400 2000 50  0001 C CNN
@@
 AR Path="/62EB4C8F/62FD0748" Ref="Q2"  Part="1"
 F 0 "Q2" V 8750 2050 50  0000 L CNN
-F 1 "PMOS" V 8600 1750 50  0000 L CNN
+F 1 "PMOS" V 8650 1750 50  0000 L CNN
 F 2 "Package_TO_SOT_SMD:SOT-23" H 9050 2100 50  0001 C CNN
 F 3 "~" H 8850 2000 50  0001 C CNN
@@
 AR Path="/62EB4C8F/62FD074F" Ref="Q1"  Part="1"
 F 0 "Q1" V 8200 2050 50  0000 L CNN
-F 1 "PMOS" V 8050 1750 50  0000 L CNN
+F 1 "PMOS" V 8100 1750 50  0000 L CNN
 F 2 "Package_TO_SOT_SMD:SOT-23" H 8500 2100 50  0001 C CNN
 F 3 "~" H 8300 2000 50  0001 C CNN
@@
 Text Label 950  3350 2    50   ~ 0
 7SEG_B
+$Comp
+L Device:R R16
+U 1 1 5FD6D30E
+P 10050 1550
+F 0 "R16" V 9950 1550 50  0000 C CNN
+F 1 "1K" V 10050 1550 50  0000 C CNN
+F 2 "Resistor_SMD:R_0402_1005Metric" V 9980 1550 50  0001 C CNN
+F 3 "~" H 10050 1550 50  0001 C CNN
+	1    10050 1550
+	-1   0    0    1
+$EndComp
+$Comp
+L Device:R R13
+U 1 1 5FD6F24D
+P 8400 1550
+F 0 "R13" V 8300 1550 50  0000 C CNN
+F 1 "1K" V 8400 1550 50  0000 C CNN
+F 2 "Resistor_SMD:R_0402_1005Metric" V 8330 1550 50  0001 C CNN
+F 3 "~" H 8400 1550 50  0001 C CNN
+	1    8400 1550
+	-1   0    0    1
+$EndComp
+$Comp
+L Device:R R14
+U 1 1 5FD7107F
+P 8950 1550
+F 0 "R14" V 8850 1550 50  0000 C CNN
+F 1 "1K" V 8950 1550 50  0000 C CNN
+F 2 "Resistor_SMD:R_0402_1005Metric" V 8880 1550 50  0001 C CNN
+F 3 "~" H 8950 1550 50  0001 C CNN
+	1    8950 1550
+	-1   0    0    1
+$EndComp
+$Comp
+L Device:R R15
+U 1 1 5FD710FF
+P 9500 1550
+F 0 "R15" V 9400 1550 50  0000 C CNN
+F 1 "1K" V 9500 1550 50  0000 C CNN
+F 2 "Resistor_SMD:R_0402_1005Metric" V 9430 1550 50  0001 C CNN
+F 3 "~" H 9500 1550 50  0001 C CNN
+	1    9500 1550
+	-1   0    0    1
+$EndComp
+$Comp
+L Device:R R20
+U 1 1 5FD72A3D
+P 8400 2500
+F 0 "R20" V 8300 2500 50  0000 C CNN
+F 1 "1K" V 8400 2500 50  0000 C CNN
+F 2 "Resistor_SMD:R_0402_1005Metric" V 8330 2500 50  0001 C CNN
+F 3 "~" H 8400 2500 50  0001 C CNN
+	1    8400 2500
+	-1   0    0    1
+$EndComp
+$Comp
+L Device:R R34
+U 1 1 5FD72E69
+P 8950 2500
+F 0 "R34" V 8850 2500 50  0000 C CNN
+F 1 "1K" V 8950 2500 50  0000 C CNN
+F 2 "Resistor_SMD:R_0402_1005Metric" V 8880 2500 50  0001 C CNN
+F 3 "~" H 8950 2500 50  0001 C CNN
+	1    8950 2500
+	-1   0    0    1
+$EndComp
+$Comp
+L Device:R R36
+U 1 1 5FD74719
+P 9500 2500
+F 0 "R36" V 9400 2500 50  0000 C CNN
+F 1 "1K" V 9500 2500 50  0000 C CNN
+F 2 "Resistor_SMD:R_0402_1005Metric" V 9430 2500 50  0001 C CNN
+F 3 "~" H 9500 2500 50  0001 C CNN
+	1    9500 2500
+	-1   0    0    1
+$EndComp
+$Comp
+L Device:R R37
+U 1 1 5FD747A1
+P 10050 2500
+F 0 "R37" V 9950 2500 50  0000 C CNN
+F 1 "1K" V 10050 2500 50  0000 C CNN
+F 2 "Resistor_SMD:R_0402_1005Metric" V 9980 2500 50  0001 C CNN
+F 3 "~" H 10050 2500 50  0001 C CNN
+	1    10050 2500
+	-1   0    0    1
+$EndComp
+Wire Wire Line
+	8300 1700 8400 1700
+Wire Wire Line
+	8850 1700 8950 1700
+Wire Wire Line
+	9400 1700 9500 1700
+Wire Wire Line
+	9950 1700 10050 1700
+Wire Wire Line
+	8300 2650 8400 2650
+Wire Wire Line
+	8850 2650 8950 2650
+Wire Wire Line
+	9400 2650 9500 2650
+Wire Wire Line
+	9950 2650 10050 2650
+$Comp
+L power:+3.3V #PWR?
+U 1 1 5FD90105
+P 9500 2350
+AR Path="/5FD90105" Ref="#PWR?"  Part="1"
+AR Path="/62EB4C8F/5FD90105" Ref="#PWR0129"  Part="1"
+F 0 "#PWR0129" H 9500 2200 50  0001 C CNN
+F 1 "+3.3V" V 9600 2400 50  0000 C CNN
+F 2 "" H 9500 2350 50  0001 C CNN
+F 3 "" H 9500 2350 50  0001 C CNN
+	1    9500 2350
+	1    0    0    -1
+$EndComp
+$Comp
+L power:+3.3V #PWR?
+U 1 1 5FDA0B28
+P 10050 2350
+AR Path="/5FDA0B28" Ref="#PWR?"  Part="1"
+AR Path="/62EB4C8F/5FDA0B28" Ref="#PWR0130"  Part="1"
+F 0 "#PWR0130" H 10050 2200 50  0001 C CNN
+F 1 "+3.3V" V 10150 2400 50  0000 C CNN
+F 2 "" H 10050 2350 50  0001 C CNN
+F 3 "" H 10050 2350 50  0001 C CNN
+	1    10050 2350
+	1    0    0    -1
+$EndComp
+$Comp
+L power:+3.3V #PWR?
+U 1 1 5FDA0B93
+P 8950 2350
+AR Path="/5FDA0B93" Ref="#PWR?"  Part="1"
+AR Path="/62EB4C8F/5FDA0B93" Ref="#PWR0131"  Part="1"
+F 0 "#PWR0131" H 8950 2200 50  0001 C CNN
+F 1 "+3.3V" V 9050 2400 50  0000 C CNN
+F 2 "" H 8950 2350 50  0001 C CNN
+F 3 "" H 8950 2350 50  0001 C CNN
+	1    8950 2350
+	1    0    0    -1
+$EndComp
+$Comp
+L power:+3.3V #PWR?
+U 1 1 5FDA0BFE
+P 8400 2350
+AR Path="/5FDA0BFE" Ref="#PWR?"  Part="1"
+AR Path="/62EB4C8F/5FDA0BFE" Ref="#PWR0132"  Part="1"
+F 0 "#PWR0132" H 8400 2200 50  0001 C CNN
+F 1 "+3.3V" V 8500 2400 50  0000 C CNN
+F 2 "" H 8400 2350 50  0001 C CNN
+F 3 "" H 8400 2350 50  0001 C CNN
+	1    8400 2350
+	1    0    0    -1
+$EndComp
+$Comp
+L power:+3.3V #PWR?
+U 1 1 5FDA0C69
+P 8400 1400
+AR Path="/5FDA0C69" Ref="#PWR?"  Part="1"
+AR Path="/62EB4C8F/5FDA0C69" Ref="#PWR0133"  Part="1"
+F 0 "#PWR0133" H 8400 1250 50  0001 C CNN
+F 1 "+3.3V" V 8500 1450 50  0000 C CNN
+F 2 "" H 8400 1400 50  0001 C CNN
+F 3 "" H 8400 1400 50  0001 C CNN
+	1    8400 1400
+	1    0    0    -1
+$EndComp
+$Comp
+L power:+3.3V #PWR?
+U 1 1 5FDA1934
+P 8950 1400
+AR Path="/5FDA1934" Ref="#PWR?"  Part="1"
+AR Path="/62EB4C8F/5FDA1934" Ref="#PWR0134"  Part="1"
+F 0 "#PWR0134" H 8950 1250 50  0001 C CNN
+F 1 "+3.3V" V 9050 1450 50  0000 C CNN
+F 2 "" H 8950 1400 50  0001 C CNN
+F 3 "" H 8950 1400 50  0001 C CNN
+	1    8950 1400
+	1    0    0    -1
+$EndComp
+$Comp
+L power:+3.3V #PWR?
+U 1 1 5FDA199F
+P 9500 1400
+AR Path="/5FDA199F" Ref="#PWR?"  Part="1"
+AR Path="/62EB4C8F/5FDA199F" Ref="#PWR0135"  Part="1"
+F 0 "#PWR0135" H 9500 1250 50  0001 C CNN
+F 1 "+3.3V" V 9600 1450 50  0000 C CNN
+F 2 "" H 9500 1400 50  0001 C CNN
+F 3 "" H 9500 1400 50  0001 C CNN
+	1    9500 1400
+	1    0    0    -1
+$EndComp
+$Comp
+L power:+3.3V #PWR?
+U 1 1 5FDA1A0A
+P 10050 1400
+AR Path="/5FDA1A0A" Ref="#PWR?"  Part="1"
+AR Path="/62EB4C8F/5FDA1A0A" Ref="#PWR0136"  Part="1"
+F 0 "#PWR0136" H 10050 1250 50  0001 C CNN
+F 1 "+3.3V" V 10150 1450 50  0000 C CNN
+F 2 "" H 10050 1400 50  0001 C CNN
+F 3 "" H 10050 1400 50  0001 C CNN
+	1    10050 1400
+	1    0    0    -1
+$EndComp
 $EndSCHEMATC
