File: dsky/dsky-MCU.sch (KiCad schematic (older format))
At the start: 27 parts, among them J1 USB_B_Micro, J2 Conn_ARM_JTAG_SWD_10, SW1 SW_DPST, U1 STM32F407VGTx, Y1 25MHz

Commit message: this hard drive is dying
Parts:
- C1, C2, C3, C4, C5, C6, C7: footprint Capacitor_SMD:C_0603_1608Metric -> Capacitor_SMD:C_0402_1005Metric
- R1, R2, R3, R4: footprint Resistor_SMD:R_0603_1608Metric -> Resistor_SMD:R_0402_1005Metric
Connections:
- net KEY_IRQ: now also U1.18 (PC3); no longer U1.95 (PB8)
- net LED_BLANK: now reaches U1.78 (PC10)
- net LED_LATCH: now reaches U1.79 (PC11)
- net LED_MTX_SDB: no longer names the net of U1.91 (PB5)
Other:
- moved on the sheet: C13, C14, J2, JP2, JP3, JP4, R3, R4, Y1
