File: dsky/dsky-ext-flash.sch (KiCad schematic (older format))
At the start: 6 parts, among them J18 EXT_FLASH_PROG, U29 W25Q80DV

Commit message: this hard drive is dying
Parts:
- C35: footprint Capacitor_SMD:C_0603_1608Metric -> Capacitor_SMD:C_0402_1005Metric
- R28, R29, R30: footprint Resistor_SMD:R_0603_1608Metric -> Resistor_SMD:R_0402_1005Metric
- U29: footprint (none) -> Package_SO:SOIJ-8_5.3x5.3mm_P1.27mm
Changed lines of the file:
@@
 F 0 "U29" H 5850 4325 50  0000 C CNN
 F 1 "W25Q80DV" H 5850 4234 50  0000 C CNN
-F 2 "" H 5900 3650 50  0001 C CNN
+F 2 "Package_SO:SOIJ-8_5.3x5.3mm_P1.27mm" H 5900 3650 50  0001 C CNN
 F 3 "" H 5900 3650 50  0001 C CNN
 	1    5850 3650
@@
 F 0 "C35" H 6535 3804 50  0000 R CNN
 F 1 "100nF" H 6535 3895 50  0000 R CNN
-F 2 "Capacitor_SMD:C_0603_1608Metric" H 6688 3700 50  0001 C CNN
+F 2 "Capacitor_SMD:C_0402_1005Metric" H 6688 3700 50  0001 C CNN
 F 3 "~" H 6650 3850 50  0001 C CNN
 	1    6650 3850
@@
 F 0 "R28" H 7070 3346 50  0000 L CNN
 F 1 "1K" H 7070 3255 50  0000 L CNN
-F 2 "Resistor_SMD:R_0603_1608Metric" V 6930 3300 50  0001 C CNN
+F 2 "Resistor_SMD:R_0402_1005Metric" V 6930 3300 50  0001 C CNN
 F 3 "~" H 7000 3300 50  0001 C CNN
 	1    7000 3300
@@
 F 0 "R30" H 4220 3496 50  0000 L CNN
 F 1 "1K" H 4220 3405 50  0000 L CNN
-F 2 "Resistor_SMD:R_0603_1608Metric" V 4080 3450 50  0001 C CNN
+F 2 "Resistor_SMD:R_0402_1005Metric" V 4080 3450 50  0001 C CNN
 F 3 "~" H 4150 3450 50  0001 C CNN
 	1    4150 3450
@@
 F 0 "R29" H 3970 3496 50  0000 L CNN
 F 1 "1K" H 3970 3405 50  0000 L CNN
-F 2 "Resistor_SMD:R_0603_1608Metric" V 3830 3450 50  0001 C CNN
+F 2 "Resistor_SMD:R_0402_1005Metric" V 3830 3450 50  0001 C CNN
 F 3 "~" H 3900 3450 50  0001 C CNN
 	1    3900 3450
