File: dsky/dsky-keys.sch (KiCad schematic (older format))
At the start: 42 parts, among them J10 Conn_01x01, J11 Conn_01x01, J12 Conn_01x01, J13 Conn_01x01, J14 Conn_01x01, J15 Conn_01x01, J16 Conn_01x01, J17 Conn_01x01, J3 Conn_01x01, J4 Conn_01x01, J5 Conn_01x01, J6 Conn_01x01, J7 Conn_01x01, J8 Conn_01x01, J9 Conn_01x01, SW3 SW_SPST, SW4 SW_SPST, SW5 SW_SPST, SW6 SW_SPST, SW7 SW_SPST, U28 BS8116A-3

Commit message: this hard drive is dying
Parts:
- C19, C20, C21, C22, C23, C24, C25, C26, C28, C29, C30, C31, C32, C33, C34: footprint Capacitor_SMD:C_0402_1005Metric -> Capacitor_SMD:C_0603_1608Metric
- C27: footprint Capacitor_SMD:C_0603_1608Metric -> Capacitor_SMD:C_0402_1005Metric
- R23, R24, R25, R26, R27: footprint Resistor_SMD:R_0603_1608Metric -> Resistor_SMD:R_0402_1005Metric
- U28: footprint (none) -> Package_SO:SOIC-20W_7.5x12.8mm_P1.27mm
Changed lines of the file:
@@
 F 0 "U28" H 5100 4700 50  0000 C CNN
 F 1 "BS8116A-3" H 5100 4600 50  0000 C CNN
-F 2 "" H 5100 3950 50  0001 C CNN
+F 2 "Package_SO:SOIC-20W_7.5x12.8mm_P1.27mm" H 5100 3950 50  0001 C CNN
 F 3 "" H 5100 3950 50  0001 C CNN
 	1    5100 3900
@@
 F 0 "C27" H 5785 4354 50  0000 R CNN
 F 1 "100nF" H 5785 4445 50  0000 R CNN
-F 2 "Capacitor_SMD:C_0603_1608Metric" H 5938 4250 50  0001 C CNN
+F 2 "Capacitor_SMD:C_0402_1005Metric" H 5938 4250 50  0001 C CNN
 F 3 "~" H 5900 4400 50  0001 C CNN
 	1    5900 4400
@@
 F 0 "C26" V 4650 2850 50  0000 C CNN
 F 1 "25pF" V 4750 2800 50  0000 C CNN
-F 2 "Capacitor_SMD:C_0402_1005Metric" H 4738 2800 50  0001 C CNN
+F 2 "Capacitor_SMD:C_0603_1608Metric" H 4738 2800 50  0001 C CNN
 F 3 "~" H 4700 2950 50  0001 C CNN
 	1    4700 2950
@@
 F 0 "C24" V 4650 2650 50  0000 C CNN
 F 1 "25pF" V 4750 2600 50  0000 C CNN
-F 2 "Capacitor_SMD:C_0402_1005Metric" H 4738 2600 50  0001 C CNN
+F 2 "Capacitor_SMD:C_0603_1608Metric" H 4738 2600 50  0001 C CNN
 F 3 "~" H 4700 2750 50  0001 C CNN
 	1    4700 2750
@@
 F 0 "C22" V 4650 2450 50  0000 C CNN
 F 1 "25pF" V 4750 2400 50  0000 C CNN
-F 2 "Capacitor_SMD:C_0402_1005Metric" H 4738 2400 50  0001 C CNN
+F 2 "Capacitor_SMD:C_0603_1608Metric" H 4738 2400 50  0001 C CNN
 F 3 "~" H 4700 2550 50  0001 C CNN
 	1    4700 2550
@@
 F 0 "C20" V 4650 2250 50  0000 C CNN
 F 1 "25pF" V 4750 2200 50  0000 C CNN
-F 2 "Capacitor_SMD:C_0402_1005Metric" H 4738 2200 50  0001 C CNN
+F 2 "Capacitor_SMD:C_0603_1608Metric" H 4738 2200 50  0001 C CNN
 F 3 "~" H 4700 2350 50  0001 C CNN
 	1    4700 2350
@@
 F 0 "C25" V 3900 2850 50  0000 C CNN
 F 1 "25pF" V 4000 2800 50  0000 C CNN
-F 2 "Capacitor_SMD:C_0402_1005Metric" H 3988 2800 50  0001 C CNN
+F 2 "Capacitor_SMD:C_0603_1608Metric" H 3988 2800 50  0001 C CNN
 F 3 "~" H 3950 2950 50  0001 C CNN
 	1    3950 2950
@@
 F 0 "C23" V 3900 2650 50  0000 C CNN
 F 1 "25pF" V 4000 2600 50  0000 C CNN
-F 2 "Capacitor_SMD:C_0402_1005Metric" H 3988 2600 50  0001 C CNN
+F 2 "Capacitor_SMD:C_0603_1608Metric" H 3988 2600 50  0001 C CNN
 F 3 "~" H 3950 2750 50  0001 C CNN
 	1    3950 2750
@@
 F 0 "C21" V 3900 2450 50  0000 C CNN
 F 1 "25pF" V 4000 2400 50  0000 C CNN
-F 2 "Capacitor_SMD:C_0402_1005Metric" H 3988 2400 50  0001 C CNN
+F 2 "Capacitor_SMD:C_0603_1608Metric" H 3988 2400 50  0001 C CNN
 F 3 "~" H 3950 2550 50  0001 C CNN
 	1    3950 2550
@@
 F 0 "C19" V 3900 2250 50  0000 C CNN
 F 1 "25pF" V 4000 2200 50  0000 C CNN
-F 2 "Capacitor_SMD:C_0402_1005Metric" H 3988 2200 50  0001 C CNN
+F 2 "Capacitor_SMD:C_0603_1608Metric" H 3988 2200 50  0001 C CNN
 F 3 "~" H 3950 2350 50  0001 C CNN
 	1    3950 2350
@@
 F 0 "C33" V 4650 5200 50  0000 C CNN
 F 1 "25pF" V 4750 5150 50  0000 C CNN
-F 2 "Capacitor_SMD:C_0402_1005Metric" H 4738 5150 50  0001 C CNN
+F 2 "Capacitor_SMD:C_0603_1608Metric" H 4738 5150 50  0001 C CNN
 F 3 "~" H 4700 5300 50  0001 C CNN
 	1    4700 5300
@@
 F 0 "C31" V 4650 5000 50  0000 C CNN
 F 1 "25pF" V 4750 4950 50  0000 C CNN
-F 2 "Capacitor_SMD:C_0402_1005Metric" H 4738 4950 50  0001 C CNN
+F 2 "Capacitor_SMD:C_0603_1608Metric" H 4738 4950 50  0001 C CNN
 F 3 "~" H 4700 5100 50  0001 C CNN
 	1    4700 5100
@@
 F 0 "C29" V 4650 4800 50  0000 C CNN
 F 1 "25pF" V 4750 4750 50  0000 C CNN
-F 2 "Capacitor_SMD:C_0402_1005Metric" H 4738 4750 50  0001 C CNN
+F 2 "Capacitor_SMD:C_0603_1608Metric" H 4738 4750 50  0001 C CNN
 F 3 "~" H 4700 4900 50  0001 C CNN
 	1    4700 4900
@@
 F 0 "C34" V 3850 5350 50  0000 C CNN
 F 1 "25pF" V 3950 5300 50  0000 C CNN
-F 2 "Capacitor_SMD:C_0402_1005Metric" H 3938 5300 50  0001 C CNN
+F 2 "Capacitor_SMD:C_0603_1608Metric" H 3938 5300 50  0001 C CNN
 F 3 "~" H 3900 5450 50  0001 C CNN
 	1    3900 5450
@@
 F 0 "C32" V 3850 5150 50  0000 C CNN
 F 1 "25pF" V 3950 5100 50  0000 C CNN
-F 2 "Capacitor_SMD:C_0402_1005Metric" H 3938 5100 50  0001 C CNN
+F 2 "Capacitor_SMD:C_0603_1608Metric" H 3938 5100 50  0001 C CNN
 F 3 "~" H 3900 5250 50  0001 C CNN
 	1    3900 5250
@@
 F 0 "C30" V 3850 4950 50  0000 C CNN
 F 1 "25pF" V 3950 4900 50  0000 C CNN
-F 2 "Capacitor_SMD:C_0402_1005Metric" H 3938 4900 50  0001 C CNN
+F 2 "Capacitor_SMD:C_0603_1608Metric" H 3938 4900 50  0001 C CNN
 F 3 "~" H 3900 5050 50  0001 C CNN
 	1    3900 5050
@@
 F 0 "C28" V 3850 4750 50  0000 C CNN
 F 1 "25pF" V 3950 4700 50  0000 C CNN
-F 2 "Capacitor_SMD:C_0402_1005Metric" H 3938 4700 50  0001 C CNN
+F 2 "Capacitor_SMD:C_0603_1608Metric" H 3938 4700 50  0001 C CNN
 F 3 "~" H 3900 4850 50  0001 C CNN
 	1    3900 4850
@@
 F 0 "R23" H 8120 3496 50  0000 L CNN
 F 1 "1K" V 8050 3400 50  0000 L CNN
-F 2 "Resistor_SMD:R_0603_1608Metric" V 7980 3450 50  0001 C CNN
+F 2 "Resistor_SMD:R_0402_1005Metric" V 7980 3450 50  0001 C CNN
 F 3 "~" H 8050 3450 50  0001 C CNN
 	1    8050 3450
@@
 F 0 "R24" H 8120 3896 50  0000 L CNN
 F 1 "1K" V 8050 3800 50  0000 L CNN
-F 2 "Resistor_SMD:R_0603_1608Metric" V 7980 3850 50  0001 C CNN
+F 2 "Resistor_SMD:R_0402_1005Metric" V 7980 3850 50  0001 C CNN
 F 3 "~" H 8050 3850 50  0001 C CNN
 	1    8050 3850
@@
 F 0 "R25" H 8120 4296 50  0000 L CNN
 F 1 "1K" V 8050 4200 50  0000 L CNN
-F 2 "Resistor_SMD:R_0603_1608Metric" V 7980 4250 50  0001 C CNN
+F 2 "Resistor_SMD:R_0402_1005Metric" V 7980 4250 50  0001 C CNN
 F 3 "~" H 8050 4250 50  0001 C CNN
 	1    8050 4250
@@
 F 0 "R26" H 8120 4696 50  0000 L CNN
 F 1 "1K" V 8050 4600 50  0000 L CNN
-F 2 "Resistor_SMD:R_0603_1608Metric" V 7980 4650 50  0001 C CNN
+F 2 "Resistor_SMD:R_0402_1005Metric" V 7980 4650 50  0001 C CNN
 F 3 "~" H 8050 4650 50  0001 C CNN
 	1    8050 4650
@@
 F 0 "R27" H 8120 5096 50  0000 L CNN
 F 1 "1K" V 8050 5000 50  0000 L CNN
-F 2 "Resistor_SMD:R_0603_1608Metric" V 7980 5050 50  0001 C CNN
+F 2 "Resistor_SMD:R_0402_1005Metric" V 7980 5050 50  0001 C CNN
 F 3 "~" H 8050 5050 50  0001 C CNN
 	1    8050 5050
